File: hardware/rainpoint_carrier/kicad/rainpoint_carrier.kicad_pcb (KiCad board)
At the start: 2 copper layers, 68 x 66 mm, 9 parts, among them J1 ESP32_Left_1x15, J2 ESP32_Right_1x15, J3 CC1101_2x4

Commit message: Preserve unfinished Rev B carrier design for later physical review
Parts:
- moved C2 15.0 mm to (146.5, 74.0)
- moved C1 9.00 mm to (146.5, 77.0)
- moved J3 7.62 mm to (141.0, 79.2)
Routing:
- net /3V3: track 34.4 -> 83.7 mm, vias 0 -> 1
- net /RADIO_GDO2: track 125.7 -> 118.1 mm, vias 0 -> 1
- net /RADIO_MISO: track 7.55 -> 12.6 mm
- net /RADIO_MOSI: track 21.1 -> 24.6 mm
- net /RADIO_GDO0: track 84.7 -> 87.2 mm
- net /RADIO_CSN: track 105.6 -> 108.1 mm
- net /RADIO_SCK: track 7.53 -> 7.32 mm, vias 0 -> 2
Other:
- board text added: "1 GND"
- board text added: "1 GND / 2 3V3"
- board text added: "2 3V3"
- board text added: "3 GDO0"
- board text added: "4 CSN"
- board text added: "5 SCK"
- board text added: "6 MOSI"
- board text added: "7 MISO"
- board text added: "8 GDO2"
- board text added: "RAINPOINT RADIO NODE - REV B"
- board text removed: "RAINPOINT RADIO NODE - REV A"
